File: imac-pcb.sch (KiCad schematic (older format))
At the start: 62 parts, among them J1 EXT_IN, J2 STEREO_OUT, P1 PROBE1, P2 PATCHBAY_IO, P3 PROBE2, P4 EXT_OUT, P5 INPUTS, P6 PATCHBAY_A, P7 PWR_X3, P8 ARDUINO_MICRO, Q1 NX3008N***, Q2 PMV48XP, Q3 NX3008N***, Q4 NX3008N***, U1 MCP6004, U2 MCP6004, U3 NCP4620, U4 ADG849

Commit message: major work on PCB layout
Parts:
- removed P8: ARDUINO_MICRO, Imac:Arduino_Micro_2x1x17, symbol ARDUINO_MICRO
- removed unit 2 of U2
- added C14, C17: 1u, Capacitors_SMD:C_0805, symbol C_Small
- added C15, C16, C19, C20: 100n, Capacitors_SMD:C_0805, symbol C_Small
- added C18: 22u, Imac:2917C, symbol CP
- added D5: CLP6B-WKW, Imac:PLCC6-3in1-SMD-LED, symbol CLP6B-WKW
- added R19: 27****, Resistors_SMD:R_1812_HandSoldering, symbol R
- added SW1: RESET_SW, Imac:EVQ_BUT, symbol SW_PUSH_SMALL_H
- added unit 2 of U2
- added U5: arduino_pro_micro, Imac:arduino_pro_micro, symbol arduino_pro_micro
- added U6: NCP1117-5, TO_SOT_Packages_SMD:SOT-223, symbol AP111750
- C6: footprint Capacitors_SMD:C_0805 -> Capacitors_SMD:C_0805_HandSoldering
- Q1, Q3, Q4: footprint TO_SOT_Packages_SMD:SC-70 -> imac:SC-70-BIG-PADS
- R1, R10, R14, R15, R16, R3, R4, R5, R6, R7, R8: footprint Resistors_SMD:R_0603 -> Resistors_SMD:R_0805
- R11: value 27 -> 27****; footprint Resistors_SMD:R_1812 -> Resistors_SMD:R_1812_HandSoldering
- R12, R17, R18, R2, R9: footprint Resistors_SMD:R_0603_HandSoldering -> Resistors_SMD:R_0805_HandSoldering
- U2: value MCP6004 -> MCP6002; footprint Housings_SOIC:SOIC-14_3.9x8.7mm_Pitch1.27mm -> Imac:SOIC-8_3.9x4.9mm_Pitch1.27mm_handsolder; symbol MCP6004 -> MCP6002
Connections:
- net 12V_IN: now also C14.1, C15.1, C18.1, U6.3 (VI)
- net 5V_SYS: now also D3.1 (A1), D3.2 (A2), D3.3 (A3), D4.1 (A1), D4.2 (A2), D4.3 (A3), U2.8 (V+), C16.1, C17.1, C19.1, C20.1, D5.1 (A1), D5.2 (A2), D5.3 (A3), U2.8 (V+), U5.21 (VCC), U6.2 (VO), U6.4 (VO); no longer R11.1, R13.1, U2.4 (V+)
- net A0_IN: now also U5.17 (A0)
- net A1_IN: now also U5.18 (A1)
- net A2_IN: now also U5.19 (A2)
- net D3: now also U5.6 (D3)
- net D6: now also U5.9 (D6)
- net GND: now also U2.4 (V-), C14.2, C15.2, C16.2, C17.2, C18.2, C19.2, C20.2, SW1.1, U2.4 (V-), U5.23 (GND), U5.3 (GND), U5.4 (GND), U6.1 (GND/ADJ); no longer U2.11 (V-)
- net SWA_COM: now also P6.4 (P4), P6.5 (P5), P6.6 (P6); no longer P6.1 (P1), P6.2 (P2), P6.3 (P3)
- net SWA_NC: now also P6.7 (P7), P6.8 (P8), P6.9 (P9); no longer P6.4 (P4), P6.5 (P5), P6.6 (P6)
- net SWA_NO: now also P6.1 (P1), P6.2 (P2), P6.3 (P3); no longer P6.7 (P7), P6.8 (P8), P6.9 (P9)
- net at C12.1, R14.1: now also U2.5 (+)
- net at C13.2: now also U2.6 (-), U2.7
- net at RV1.2: now also U1.5 (+); no longer U1.3 (+)
- net at C4.1, R4.1: now also U1.3 (+); no longer U1.10 (+)
- net at C2.1, C7.2: now also U1.1, U1.2 (-); no longer U1.8, U1.9 (-)
- net at RV2.2: now also U1.10 (+); no longer U1.5 (+)
- net at D4.4 (C3), D4.5 (C2), D4.6 (C1): now also R13.1; no longer Q3.3 (D)
- net at D3.4 (C3), D3.5 (C2), D3.6 (C1): now also R11.1; no longer Q1.3 (D)
- new net: RV3.1, U1.6 (-), U1.7
- new net: RV4.1, U1.8, U1.9 (-)
- new net: Q3.3 (D), R13.2
- new net: Q1.3 (D), R11.2, R19.2
- new net: D5.4 (C3), D5.5 (C2), D5.6 (C1), R19.1
- new net: SW1.2, U5.22 (!RST)
- no-connect marks 23 -> 14
Other:
- note added: "* Resistors are optional. Can be connected with a solder bridge.\n** Trimmer can be swapped for 1meg for higher input impedance\n*** Replace/Experiment with BC817, and larger base/gate resistors\n**** Choose one LED front or back"
- note added: "5V System Regulation"
- note removed: "* Resistors are optional. Can be connected with a solder bridge.\n** Trimmer can be swapped for 1meg for higher input impedance\n*** Replace/Experiment with BC817, and larger base/gate resistors"
- moved on the sheet: C10, C11, C9, D2, D3, D4, Q1, R10, R11, R13, R9, U3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
